File: Esquematicos/CircuiteriaESP32/CircuiteriaESP32.kicad_sch (KiCad schematic)
At the start: 21 parts

Commit message: 18 abril 2023
Parts:
- added SIM800HAlim: Conn_01x01, symbol Connector_Generic:Conn_01x01
- added SIM800HControl: Conn_01x12, symbol Connector_Generic:Conn_01x12
Connections:
- net +3V3: now also SIM800HControl.1 (Pin_1)
- net +5V: now also SIM800HAlim.1 (Pin_1)
- net GND: now also SIM800HControl.11 (Pin_11), SIM800HControl.6 (Pin_6)
- net at GPSTX.1 (Pin_1): now also ESP32-2.11 (Pin_11), SIM800HControl.3 (Pin_3); no longer ESP32-2.10 (Pin_10)
Other:
- moved on the sheet: AnalogOzono, GPSTX, I2CADC1, I2CADCExterno, R2

Commit message: 4 de Mayo 2023
Parts:
- removed AlimOzono3v3: Conn_01x03, symbol Connector_Generic:Conn_01x03
- removed ESP32-1, ESP32-2: Conn_01x19, symbol Connector_Generic:Conn_01x19
- removed GPSTX: Conn_01x01, symbol Connector_Generic:Conn_01x01
- removed PuenteHAspas: Conn_01x04, symbol Connector_Generic:Conn_01x04
- added AZDeliveryESP1: ESP32-DevKitC, Espressif:ESP32-DevKitC, symbol Espressif:ESP32-DevKitC
- added Bat1+2-1, BateriaPrincipal1+2-1: Conn_01x02, Connector_PinHeader_2.54mm:PinHeader_1x02_P2.54mm_Vertical, symbol Connector_Generic:Conn_01x02
- added PuenteHAspas1: Conn_01x06, Connector_PinHeader_2.54mm:PinHeader_1x06_P2.54mm_Vertical, symbol Connector_Generic:Conn_01x06
- AlimGPS1: renamed from AlimGPS; footprint (none) -> Connector_PinHeader_2.54mm:PinHeader_1x02_P2.54mm_Vertical
- AlimOzono5V1: renamed from AlimOzono5V; footprint (none) -> Connector_PinHeader_2.54mm:PinHeader_2x03_P2.54mm_Vertical
- AnalogOzono1: renamed from AnalogOzono; footprint (none) -> Connector_PinHeader_2.54mm:PinHeader_1x03_P2.54mm_Vertical
- C1: footprint (none) -> Capacitor_THT:CP_Radial_D8.0mm_P3.50mm
- D1: renamed from D2; footprint (none) -> Diode_THT:D_5KPW_P7.62mm_Vertical_AnodeUp
- D2: renamed from D1; footprint (none) -> Diode_THT:D_5KPW_P7.62mm_Vertical_AnodeUp
- GPSUART1: renamed from UART; footprint (none) -> Connector_PinHeader_2.54mm:PinHeader_1x02_P2.54mm_Vertical
- I2CADC1: renamed from I2CADC; footprint (none) -> Connector_PinHeader_2.54mm:PinHeader_1x02_P2.54mm_Vertical
- I2CADC2: renamed from I2CADC1; footprint (none) -> Connector_PinHeader_2.54mm:PinHeader_1x02_P2.54mm_Vertical
- I2CADCExterno1: renamed from I2CADCExterno; footprint (none) -> Connector_PinHeader_2.54mm:PinHeader_1x10_P2.54mm_Vertical
- I2CTempHum1: renamed from I2CTempHum; footprint (none) -> Connector_PinHeader_2.54mm:PinHeader_2x02_P2.54mm_Vertical
- PlacaSolar1: renamed from PlacaSolar; footprint (none) -> Connector_PinHeader_2.54mm:PinHeader_1x02_P2.54mm_Vertical
- R1, R2: footprint (none) -> Resistor_THT:R_Axial_DIN0204_L3.6mm_D1.6mm_P7.62mm_Horizontal
- SIM800HAlim1: renamed from SIM800HAlim; footprint (none) -> Connector_PinHeader_2.54mm:PinHeader_1x01_P2.54mm_Vertical
- SIM800HControl1: renamed from SIM800HControl; footprint (none) -> Connector_PinHeader_2.54mm:PinHeader_1x12_P2.54mm_Vertical
- ServoExt1: renamed from ServoExt; footprint (none) -> Connector_PinHeader_2.54mm:PinHeader_1x03_P2.54mm_Vertical
- ServoInt1: renamed from ServoInt; footprint (none) -> Connector_PinHeader_2.54mm:PinHeader_1x03_P2.54mm_Vertical
Connections:
- net +5V: now also AZDeliveryESP1.19 (5V), BateriaPrincipal1+2-1.1 (Pin_1); no longer D1.1 (K), ServoExt1.2 (Pin_2), ServoInt1.2 (Pin_2)
- net GND: now also AZDeliveryESP1.38 (GND), BateriaPrincipal1+2-1.2 (Pin_2); no longer ServoExt1.3 (Pin_3), ServoInt1.3 (Pin_3)
- net at SIM800HControl1.3 (Pin_3): now also AZDeliveryESP1.28 (GPIO17)
- net at D1.2 (A), D2.2 (A), PlacaSolar1.1 (Pin_1): now also AZDeliveryESP1.8 (32K_XN/GPIO33/ADC1_CH5)
- net at AlimGPS1.2 (Pin_2): now also AZDeliveryESP1.32 (GND)
- net at ServoExt1.1 (Pin_1): now also AZDeliveryESP1.30 (GPIO18)
- net at I2CADC1.1 (Pin_1), I2CTempHum1.1 (Pin_1), R2.1: now also AZDeliveryESP1.26 (ADC2_CH0/GPIO4)
- net at I2CADC1.2 (Pin_2), I2CTempHum1.2 (Pin_2), R1.1: now also AZDeliveryESP1.23 (*MTDO/GPIO15/ADC2_CH3)
- net at AlimOzono5V1.4 (Pin_4), AlimOzono5V1.5 (Pin_5), AlimOzono5V1.6 (Pin_6)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: now also AZDeliveryESP1.14 (GND)
- net at GPSUART1.2 (Pin_2): now also AZDeliveryESP1.34 (U0RXD/GPIO3)
- net at ServoInt1.1 (Pin_1): now also AZDeliveryESP1.31 (GPIO19)
- net +3V3: no longer names the net of AlimGPS1.1 (Pin_1), I2CTempHum1.4 (Pin_4), R1.2, R2.2, SIM800HControl1.1 (Pin_1)
- net +3V3: now also AZDeliveryESP1.1 (3V3)
- new net: AZDeliveryESP1.33 (GPIO21), PuenteHAspas1.1 (Pin_1)
- new net: Bat1+2-1.2 (Pin_2), PuenteHAspas1.2 (Pin_2), PuenteHAspas1.3 (Pin_3), ServoExt1.3 (Pin_3), ServoInt1.3 (Pin_3)
- new net: Bat1+2-1.1 (Pin_1), D1.1 (K), PuenteHAspas1.4 (Pin_4), ServoExt1.2 (Pin_2), ServoInt1.2 (Pin_2)
- no-connect marks 0 -> 38
Other:
- company: (none) -> U.P.M.
- title: (none) -> AspiradO3
- moved on the sheet: AlimGPS1, AlimOzono5V1, AnalogOzono1, C1, D1, D2, GPSUART1, I2CADC1, I2CADC2, I2CADCExterno1, I2CTempHum1, PlacaSolar1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

Commit message: Lunes 8 Mayo 2023
Parts:
- removed AlimOzono5V1: Conn_02x03_Top_Bottom, Connector_PinHeader_2.54mm:PinHeader_2x03_P2.54mm_Vertical, symbol Connector_Generic:Conn_02x03_Top_Bottom
- removed I2CTempHum1: Conn_02x02_Top_Bottom, Connector_PinHeader_2.54mm:PinHeader_2x02_P2.54mm_Vertical, symbol Connector_Generic:Conn_02x02_Top_Bottom
- added AlimOzono5V1: Conn_02x03_Odd_Even, Connector_PinHeader_2.54mm:PinHeader_2x03_P2.54mm_Vertical, symbol Connector_Generic:Conn_02x03_Odd_Even
- added I2CTempHum1: Conn_02x02_Odd_Even, Connector_PinHeader_2.54mm:PinHeader_2x02_P2.54mm_Vertical, symbol Connector_Generic:Conn_02x02_Odd_Even
Connections:
- net +5V: now also AlimOzono5V1.1 (Pin_1), AlimOzono5V1.3 (Pin_3), AlimOzono5V1.5 (Pin_5)
- net GND: now also I2CTempHum1.2 (Pin_2)
- net at AZDeliveryESP1.1 (3V3), AlimGPS1.1 (Pin_1), R1.2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: now also I2CTempHum1.4 (Pin_4)
- net at AZDeliveryESP1.26 (ADC2_CH0/GPIO4), I2CADC1.1 (Pin_1), R2.1: now also I2CTempHum1.1 (Pin_1)
- net at AZDeliveryESP1.23 (*MTDO/GPIO15/ADC2_CH3), I2CADC1.2 (Pin_2), R1.1: now also I2CTempHum1.3 (Pin_3)
- net at AZDeliveryESP1.14 (GND), PlacaSolar1.2 (Pin_2): now also AlimOzono5V1.2 (Pin_2), AlimOzono5V1.4 (Pin_4), AlimOzono5V1.6 (Pin_6)

Commit message: 9 mayo 2023
Parts:
- D1, D2: footprint Diode_THT:D_5KPW_P7.62mm_Vertical_AnodeUp -> Diode_THT:D_T-1_P2.54mm_Vertical_AnodeUp
Changed lines of the file:
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@@
       (effects (font (size 1.27 1.27)))
     )
-    (property "Footprint" "Diode_THT:D_5KPW_P7.62mm_Vertical_AnodeUp" (at 33.02 62.23 0)
+    (property "Footprint" "Diode_THT:D_T-1_P2.54mm_Vertical_AnodeUp" (at 33.02 62.23 0)
       (effects (font (size 1.27 1.27)) hide)
     )
@@
       (effects (font (size 1.27 1.27)))
     )
-    (property "Footprint" "Diode_THT:D_5KPW_P7.62mm_Vertical_AnodeUp" (at 33.02 46.99 0)
-      (effects (font (size 1.27 1.27)) hide)
-    )
+    (property "Footprint" "Diode_THT:D_T-1_P2.54mm_Vertical_AnodeUp" (at 33.02 46.99 0)
+      (effects (font (size 1.27 1.27)) hide)
+    )
