File: Esquematicos/CircuiteriaESP32/CircuiteriaESP32.kicad_pcb (KiCad board)
At the start: 2 copper layers, 60 x 60 mm, 22 parts

Commit message: 9 mayo 2023
Parts:
- D1, D2: footprint Diode_THT:D_5KPW_P7.62mm_Vertical_AnodeUp -> Diode_THT:D_T-1_P2.54mm_Vertical_AnodeUp
- moved PlacaSolar1 7.82 mm to (83.0, 147.8), turned to -90 degrees
- moved SIM800HAlim1 5.35 mm to (80.5, 166.2)
- moved AlimOzono5V1 3.25 mm to (80.5, 153.0)
- moved D1 2.00 mm to (81.8, 180.5)
Routing:
- net Net-(AZDeliveryESP1-32K_XN/GPIO33/ADC1_CH5): track 58.3 -> 52.0 mm
- net +5V: track 107.7 -> 105.4 mm
- net Net-(Bat1+2-1-Pin_1): track 81.4 -> 80.3 mm
- net Net-(AlimOzono5V1-Pin_2): track 20.8 -> 21.6 mm
- net Net-(AZDeliveryESP1-GPIO17): track 36.9 -> 36.2 mm
- net Net-(AZDeliveryESP1-3V3): track 92.9 -> 92.3 mm

Commit message: 10 mayo 2023
Parts:
- added G***: LOGO, LOGOS:ETSISI_logo, F.Cu at (99.0, 138.2)
